File: kicad-git-example.kicad_sch (KiCad schematic)
At the start: 6 parts, among them J1 Conn_01x20, J2 Conn_01x20, J3 Conn_01x20, J4 Conn_01x20, U1 74LS181, U2 74LS181

Commit message: Version 2
Other:
- note added: "Version 2"
Changed lines of the file:
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@@
 	(generator_version "10.0")
 	(paper "A4")
+	(text "Version 2"
+		(exclude_from_sim no)
+		(at 196.85 149.606 0)
+		(effects
+			(font
+				(size 3.81 3.81)
+			)
+		)
+	)
 	(wire
 		(pts
